File: MegaDrivePadTest.kicad_pcb (KiCad board)
At the start: 2 copper layers, 45.7 x 52.7 mm, 25 parts, among them J1 USB_B_Micro, J2 DE9_Receptacle_MountingHoles, J3 ALT POWER, SW1 SELECT

Commit message: Move USB port to edge of PCB.
Parts:
- moved J1 1.27 mm to (119.4, 85.1)
- moved J3 1.02 mm to (114.3, 93.5)
- moved R13 1.02 mm to (121.9, 93.5)
- moved R14 1.02 mm to (147.3, 93.5)
Routing:
- net GND: track 3.76 -> 12.9 mm
- net VCC: track 119.6 -> 122.4 mm
- net Net-(SW1-A): track 17.3 -> 16.3 mm
Other:
- board text added: "https://github.com/Board-Folk/MegaDrivePadTest"
Changed lines of the file:
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@@
 	)
 	(setup
+		(stackup
+			(layer "F.SilkS"
+				(type "Top Silk Screen")
+			)
+			(layer "F.Paste"
+				(type "Top Solder Paste")
+			)
+			(layer "F.Mask"
+				(type "Top Solder Mask")
+				(thickness 0.01)
+			)
+			(layer "F.Cu"
+				(type "copper")
+				(thickness 0.035)
+			)
+			(layer "dielectric 1"
+				(type "core")
+				(thickness 1.51)
+				(material "FR4")
+				(epsilon_r 4.5)
+				(loss_tangent 0.02)
+			)
+			(layer "B.Cu"
+				(type "copper")
+				(thickness 0.035)
+			)
+			(layer "B.Mask"
+				(type "Bottom Solder Mask")
+				(thickness 0.01)
+			)
+			(layer "B.Paste"
+				(type "Bottom Solder Paste")
+			)
+			(layer "B.SilkS"
+				(type "Bottom Silk Screen")
+			)
+			(copper_finish "None")
+			(dielectric_constraints no)
+		)
 		(pad_to_mask_clearance 0)
 		(allow_soldermask_bridges_in_footprints no)
@@
 	(footprint "Connector_PinHeader_2.54mm:PinHeader_1x02_P2.54mm_Vertical"
 		(layer "F.Cu")
-		(at 114.3 94.488 90)
+		(at 114.3 93.472 90)
 		(descr "Through hole straight pin header, 1x02, 2.54mm pitch, single row")
 		(tags "Through hole pin header THT 1x02 2.54mm single row")
@@
 	(footprint "Connector_USB:USB_Micro-B_Amphenol_10103594-0001LF_Horizontal"
 		(layer "F.Cu")
-		(at 119.38 86.36 180)
+		(at 119.38 85.09 180)
 		(descr "Micro USB Type B 10103594-0001LF, http://cdn.amphenol-icc.com/media/wysiwyg/files/drawing/10103594.pdf")
 		(tags "USB USB_B USB_micro USB_OTG")
@@
 	(footprint "MegaDrivePadTest_Library:R_Combo"
 		(layer "F.Cu")
-		(at 147.32 94.488 180)
+		(at 147.32 93.472 180)
 		(descr "Resistor, Axial_DIN0207 series, Axial, Horizontal, pin pitch=10.16mm, 0.25W = 1/4W, length*diameter=6.3*2.5mm^2, http://cdn-reichelt.de/documents/datenblatt/B400/1_4W%23YAG.pdf")
 		(tags "Resistor Axial_DIN0207 series Axial Horizontal pin pitch 10.16mm 0.25W = 1/4W length 6.3mm diameter 2.5mm")
@@
 	(footprint "MegaDrivePadTest_Library:R_Combo"
 		(layer "F.Cu")
-		(at 121.92 94.488)
+		(at 121.92 93.472)
 		(descr "Resistor, Axial_DIN0207 series, Axial, Horizontal, pin pitch=10.16mm, 0.25W = 1/4W, length*diameter=6.3*2.5mm^2, http://cdn-reichelt.de/documents/datenblatt/B400/1_4W%23YAG.pdf")
 		(tags "Resistor Axial_DIN0207 series Axial Horizontal pin pitch 10.16mm 0.25W = 1/4W length 6.3mm diameter 2.5mm")
@@
 		)
 	)
+	(gr_text "https://github.com/Board-Folk/MegaDrivePadTest"
+		(at 134.62 132.588 0)
+		(layer "B.SilkS")
+		(effects
+			(font
+				(size 1 1)
+				(thickness 0.15)
+			)
+			(justify mirror)
+		)
+	)
 	(gr_text "+5V"
-		(at 114.3 92.71 90)
+		(at 114.3 91.694 90)
 		(layer "F.SilkS")
 		(effects
@@
 	)
 	(gr_text "GND"
-		(at 116.84 92.71 90)
+		(at 116.84 91.694 90)
 		(layer "F.SilkS")
 		(effects
@@
 	)
 	(segment
-		(start 118.445 84.975)
-		(end 116.945 84.975)
+		(start 120.707 85.655)
+		(end 122.355 85.655)
 		(width 0.35)
 		(layer "F.Cu")
@@
 	)
 	(segment
-		(start 116.945 84.975)
-		(end 116.675 85.245)
+		(start 118.105 86.855)
+		(end 118.105 85.707)
 		(width 0.35)
 		(layer "F.Cu")
@@
 	)
 	(segment
-		(start 121.865 84.975)
-		(end 122.135 85.245)
+		(start 118.445 85.263)
+		(end 118.053 85.655)
 		(width 0.35)
 		(layer "F.Cu")
@@
 	)
 	(segment
-		(start 120.365 84.975)
-		(end 121.865 84.975)
+		(start 120.365 83.705)
+		(end 120.365 85.313)
+		(width 0.35)
+		(layer "F.Cu")
+		(net 13)
+	)
+	(segment
+		(start 122.135 83.975)
+		(end 120.635 83.975)
+		(width 0.35)
+		(layer "F.Cu")
+		(net 13)
+	)
+	(segment
+		(start 120.365 85.313)
+		(end 120.707 85.655)
+		(width 0.35)
+		(layer "F.Cu")
+		(net 13)
+	)
+	(segment
+		(start 116.675 83.975)
+		(end 118.175 83.975)
+		(width 0.35)
+		(layer "F.Cu")
+		(net 13)
+	)
+	(segment
+		(start 118.053 85.655)
+		(end 116.405 85.655)
+		(width 0.35)
+		(layer "F.Cu")
+		(net 13)
+	)
+	(segment
+		(start 118.105 85.707)
+		(end 118.053 85.655)
+		(width 0.35)
+		(layer "F.Cu")
+		(net 13)
+	)
+	(segment
+		(start 118.445 83.705)
+		(end 118.445 85.263)
+		(width 0.35)
+		(layer "F.Cu")
+		(net 13)
+	)
+	(segment
+		(start 121.865 83.705)
+		(end 122.135 83.975)
+		(width 0.35)
+		(layer "F.Cu")
+		(net 13)
+	)
+	(segment
+		(start 118.175 83.975)
+		(end 118.445 83.705)
+		(width 0.35)
+		(layer "F.Cu")
+		(net 13)
+	)
+	(segment
+		(start 120.635 83.975)
+		(end 120.365 83.705)
 		(width 0.35)
 		(layer "F.Cu")
@@
 	)
 	(segment
-		(start 151.13 92.71)
-		(end 151.13 86.0425)
+		(start 150.368 93.472)
+		(end 151.13 92.71)
 		(width 0.35)
 		(layer "F.Cu")
@@
 	)
 	(segment
-		(start 147.32 94.488)
-		(end 149.352 94.488)
+		(start 147.32 93.472)
+		(end 150.368 93.472)
 		(width 0.35)
 		(layer "F.Cu")
@@
 	)
 	(segment
-		(start 149.352 94.488)
-		(end 151.13 92.71)
+		(start 151.13 92.71)
+		(end 151.13 86.0425)
 		(width 0.35)
 		(layer "F.Cu")
@@
 	)
 	(segment
-		(start 142.24 117.475)
-		(end 144.145 119.38)
+		(start 142.24 98.552)
+		(end 142.24 117.475)
 		(width 0.35)
 		(layer "F.Cu")
@@
 	)
 	(segment
-		(start 120.705 90.115)
-		(end 119.6975 91.1225)
+		(start 120.705 89.353)
+		(end 119.888 90.17)
 		(width 0.35)
 		(layer "F.Cu")
@@
 	)
 	(segment
-		(start 142.24 99.06)
-		(end 142.24 117.475)
+		(start 114.3 90.932)
+		(end 114.3 93.472)
 		(width 0.35)
 		(layer "F.Cu")
@@
 	)
 	(segment
-		(start 114.3 92.075)
-		(end 114.3 94.488)
+		(start 131.318 96.52)
+		(end 115.03025 96.52)
 		(width 0.35)
 		(layer "F.Cu")
@@
 	)
 	(segment
-		(start 120.705 88.125)
-		(end 120.705 90.115)
+		(start 115.03025 96.52)
+		(end 114.3 95.78975)
 		(width 0.35)
 		(layer "F.Cu")
@@
 	)
 	(segment
-		(start 137.16 94.488)
-		(end 137.668 94.488)
-		(width 0.35)
-		(layer "F.Cu")
-		(net 17)
-	)
-	(segment
-		(start 115.53825 97.028)
-		(end 114.3 95.78975)
+		(start 132.08 95.758)
+		(end 131.318 96.52)
 		(width 0.35)
 		(layer "F.Cu")
@@
 	)
 	(segment
-		(start 132.08 94.488)
-		(end 132.08 95.758)
+		(start 136.525 119.38)
+		(end 140.335 119.38)
 		(width 0.35)
 		(layer "F.Cu")
@@
 	)
 	(segment
-		(start 119.6975 91.1225)
-		(end 115.2525 91.1225)
+		(start 115.062 90.17)
+		(end 114.3 90.932)
 		(width 0.35)
 		(layer "F.Cu")
@@
 	)
 	(segment
-		(start 136.525 119.38)
-		(end 140.335 119.38)
+		(start 132.08 93.472)
+		(end 137.16 93.472)
 		(width 0.35)
 		(layer "F.Cu")
@@
 	)
 	(segment
-		(start 132.08 94.488)
-		(end 137.16 94.488)
+		(start 132.715 119.38)
+		(end 121.285 119.38)
 		(width 0.35)
 		(layer "F.Cu")
@@
 	)
 	(segment
-		(start 137.668 94.488)
-		(end 142.24 99.06)
+		(start 137.16 93.472)
+		(end 142.24 98.552)
 		(width 0.35)
 		(layer "F.Cu")
@@
 	)
 	(segment
-		(start 132.08 95.758)
-		(end 130.81 97.028)
+		(start 140.335 126.825)
+		(end 140.16 127)
 		(width 0.35)
 		(layer "F.Cu")
@@
 	)
 	(segment
-		(start 132.715 119.38)
-		(end 121.285 119.38)
+		(start 113.665 119.38)
+		(end 117.475 119.38)
 		(width 0.35)
 		(layer "F.Cu")
@@
 	)
 	(segment
-		(start 140.335 126.825)
-		(end 140.16 127)
+		(start 155.575 119.38)
+		(end 151.765 119.38)
 		(width 0.35)
 		(layer "F.Cu")
@@
 	)
 	(segment
-		(start 113.665 119.38)
-		(end 117.475 119.38)
+		(start 144.145 119.38)
+		(end 147.955 119.38)
 		(width 0.35)
 		(layer "F.Cu")
@@
 	)
 	(segment
-		(start 155.575 119.38)
-		(end 151.765 119.38)
+		(start 147.955 119.38)
+		(end 140.335 119.38)
 		(width 0.35)
 		(layer "F.Cu")
@@
 	)
 	(segment
-		(start 114.3 95.78975)
-		(end 114.3 94.488)
+		(start 142.24 117.475)
+		(end 144.145 119.38)
 		(width 0.35)
 		(layer "F.Cu")
@@
 	)
 	(segment
-		(start 144.145 119.38)
-		(end 147.955 119.38)
+		(start 120.705 86.855)
+		(end 120.705 89.353)
 		(width 0.35)
 		(layer "F.Cu")
@@
 	)
 	(segment
-		(start 147.955 119.38)
-		(end 140.335 119.38)
+		(start 119.888 90.17)
+		(end 115.062 90.17)
 		(width 0.35)
 		(layer "F.Cu")
@@
 	)
 	(segment
-		(start 115.2525 91.1225)
-		(end 114.3 92.075)
+		(start 132.08 93.472)
+		(end 132.08 95.758)
 		(width 0.35)
 		(layer "F.Cu")
@@
 	)
 	(segment
-		(start 130.81 97.028)
-		(end 115.53825 97.028)
+		(start 114.3 95.78975)
+		(end 114.3 93.472)
 		(width 0.35)
 		(layer "F.Cu")
@@
 	)
 	(segment
-		(start 121.92 92.075)
-		(end 123.19 90.805)
+		(start 121.92 93.472)
+		(end 121.92 92.075)
 		(width 0.35)
 		(layer "F.Cu")
@@
 	)
 	(segment
-		(start 121.92 94.488)
-		(end 121.92 92.075)
+		(start 131.1275 90.805)
+		(end 132.08 89.8525)
 		(width 0.35)
 		(layer "F.Cu")
@@
 	)
 	(segment
-		(start 131.1275 90.805)
-		(end 132.08 89.8525)
+		(start 121.92 92.075)
+		(end 123.19 90.805)
 		(width 0.35)
 		(layer "F.Cu")
@@
 		(polygon
 			(pts
-				(xy 117.348 85.598) (xy 121.412 85.598) (xy 121.412 87.376) (xy 117.348 87.376)
+				(xy 121.666 84.836) (xy 121.666 85.852) (xy 117.094 85.852) (xy 117.094 84.836)
 			)
 		)

Commit message: Allow for wider switches.
Other:
- board text added: "JLCJLCJLCJLC"
Changed lines of the file:
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@@
 			(plot_on_all_layers_selection 0x0000000_00000000)
 			(disableapertmacros no)
-			(usegerberextensions no)
-			(usegerberattributes yes)
-			(usegerberadvancedattributes yes)
-			(creategerberjobfile yes)
+			(usegerberextensions yes)
+			(usegerberattributes no)
+			(usegerberadvancedattributes no)
+			(creategerberjobfile no)
 			(dashed_line_dash_ratio 12.000000)
 			(dashed_line_gap_ratio 3.000000)
@@
 			(plotinvisibletext no)
 			(sketchpadsonfab no)
-			(subtractmaskfromsilk no)
+			(subtractmaskfromsilk yes)
 			(outputformat 1)
 			(mirror no)
-			(drillshape 1)
+			(drillshape 0)
 			(scaleselection 1)
-			(outputdirectory "")
+			(outputdirectory "mdpadtest-gerbers-jlc")
 		)
 	)
@@
 		)
 		(property "Value" "SELECT"
-			(at 0 3.2385 0)
+			(at 0 3.8735 0)
 			(unlocked yes)
 			(layer "F.SilkS")
@@
 		(attr through_hole)
 		(fp_rect
-			(start -4 -2)
-			(end 4 2)
+			(start -5.016 -2)
+			(end 5.016 2)
 			(stroke
 				(width 0.2)
@@
 			)
 		)
-		(pad "1" thru_hole circle
-			(at -2.54 0)
-			(size 2 2)
-			(drill 1.2)
+		(pad "1" thru_hole oval
+			(at -3.048 0)
+			(size 3 2)
+			(drill oval 2.2 1.2)
 			(layers "*.Cu" "*.Mask")
 			(remove_unused_layers no)
@@
 			(pintype "passive")
 		)
-		(pad "3" thru_hole circle
-			(at 2.54 0)
-			(size 2 2)
-			(drill 1.2)
+		(pad "3" thru_hole oval
+			(at 3.048 0)
+			(size 3 2)
+			(drill oval 2.2 1.2)
 			(layers "*.Cu" "*.Mask")
 			(remove_unused_layers no)
@@
 		)
 	)
+	(gr_text "JLCJLCJLCJLC"
+		(at 134.62 132.6 0)
+		(layer "F.SilkS")
+		(effects
+			(font
+				(size 1 1)
+				(thickness 0.15)
+			)
+		)
+	)
 	(gr_text "+5V"
 		(at 114.3 91.694 90)
@@
 	)
 	(segment
-		(start 132.08 89.8525)
-		(end 132.08 86.0425)
+		(start 131.572 89.916)
+		(end 131.572 86.0425)
 		(width 0.35)
 		(layer "F.Cu")
@@
 	)
 	(segment
-		(start 123.19 90.805)
-		(end 131.1275 90.805)
+		(start 121.92 92.075)
+		(end 123.19 90.805)
 		(width 0.35)
 		(layer "F.Cu")
@@
 	)
 	(segment
-		(start 121.92 93.472)
-		(end 121.92 92.075)
+		(start 123.19 90.805)
+		(end 130.683 90.805)
 		(width 0.35)
 		(layer "F.Cu")
@@
 	)
 	(segment
-		(start 131.1275 90.805)
-		(end 132.08 89.8525)
+		(start 130.683 90.805)
+		(end 131.572 89.916)
 		(width 0.35)
 		(layer "F.Cu")
@@
 	)
 	(segment
-		(start 121.92 92.075)
-		(end 123.19 90.805)
+		(start 121.92 93.472)
+		(end 121.92 92.075)
 		(width 0.35)
 		(layer "F.Cu")
